File: hardware/periph_board/periph_board.kicad_sch (KiCad schematic)
At the start: 25 parts, among them IC100 CD74HC4067SM96, IC101 LM2937ET-3.3_NOPB, IC102 ADC121S021CIMFX_NOPB, J100 2x10 Male Pins

Commit message: Adjusted spacing to 13.5mm between hall effects
Parts:
- removed TP103: 3V3A, SamacSys_Parts:bettertestpoint2, symbol Connector:TestPoint
- removed TP110: GND, SamacSys_Parts:bettertestpoint2, symbol Connector:TestPoint
- added TP112: GND, SamacSys_Parts:bettertestpoint2, symbol Connector:TestPoint
- added TP113: 3V3A, SamacSys_Parts:bettertestpoint2, symbol Connector:TestPoint
- renumbered TP102 to TP101, TP105 to TP102, TP106 to TP103, TP107 to TP104, TP108 to TP105, TP109 to TP106, TP111 to TP107, TP112 to TP108, TP113 to TP109, TP114 to TP110, TP115 to TP111
Connections:
- net +3.3VADC: now also TP113.1
- net GND: now also TP112.1
