File: hardware/periph_board/periph_board.kicad_sch (KiCad schematic)
At the start: 45 parts, among them IC100 CD74HC4067SM96, IC101 LM2937ET-3.3_NOPB, IC102 MCP3221AxT-E_OT, J100 2x8 Socket Pins, J101 2x8 Plug Pins

Commit message: finished main pcb
Other:
- note added: "Funny LEDs"
- moved on the sheet: TP100, TP101, TP103, TP104, TP105, TP106, TP107, TP108, TP109, TP110, TP111, TP112
