File: hardware/main_board/ENCODERS_BUTTONS.kicad_sch (KiCad schematic)
At the start: 0 parts

Commit message: drew schematic
Parts:
- added J2, J3: Conn_01x05_Pin, symbol Connector:Conn_01x05_Pin
- added R6, R7: 10k, Resistor_SMD:R_0805_2012Metric, symbol Device:R_US
Connections:
- new net +3V3: J2.4 (Pin_4), J3.4 (Pin_4), R6.2, R7.2
- new net ENC1.CLK: J2.1 (Pin_1)
- new net ENC1.DT: J2.2 (Pin_2)
- new net ENC1.SW: J2.3 (Pin_3), R6.1
- new net ENC2.CLK: J3.1 (Pin_1)
- new net ENC2.DT: J3.2 (Pin_2)
- new net ENC2.SW: J3.3 (Pin_3), R7.1
- new net GND: J2.5 (Pin_5), J3.5 (Pin_5)
Other:
- note added: "Also assuming we will connect these to the board w/ wires"
- note added: "Assuming module has this layout: https://docs.wokwi.com/parts/wokwi-ky-040"
- note added: "ENC1"
- note added: "ENC2"
- note added: "Hierarchical Labels"

Commit message: save before nuke SPI ADC
Parts:
- added C5: 1u, Capacitor_SMD:C_0805_2012Metric, symbol ECE445L:C
- added IC2: SN74HC157NSR, SamacSys_Parts:SOIC127P780X200-16N, symbol SamacSys_Parts:SN74HC157NSR
Connections:
- net ENC1.CLK: now also IC2.11 (3A)
- net ENC1.DT: now also IC2.5 (2A)
- net ENC1.SW: now also IC2.2 (1A)
- net ENC2.CLK: now also IC2.10 (3B)
- net ENC2.DT: now also IC2.6 (2B)
- net ENC2.SW: now also IC2.3 (1B)
- net GND: now also C5.2, IC2.15 (~{G}), IC2.8 (GND)
- new net: C5.1, IC2.16 (VCC)
- new net ENC.CLK: IC2.9 (3Y)
- new net ENC.DT: IC2.7 (2Y)
- new net ENC.SW: IC2.4 (1Y)
- new net ENC_TOGGLE: IC2.1 (~{A}/B)
- no-connect marks 0 -> 3
Other:
- note added: "Encoder MUX"
- note added: "this is necessary bc we ran out of gpio lol idea is same as how our Hall ADC is set up except this will strobe between the two encoder inputs given a gpio clock"
- moved on the sheet: J2, J3, R6, R7
