File: hardware/main_board/P_BOARD_INT.kicad_sch (KiCad schematic)
At the start: 2 parts, among them J9 2x10 Male Pins

Commit message: drew schematic
Parts:
- removed TP7: GND, SamacSys_Parts:bettertestpoint2, symbol Connector:TestPoint
- renumbered J9 to J7

Commit message: port to i2c for both boards. periph board passes drc
Parts:
- J7: value 2x10 Male Pins -> 2x18 Male Pins
Changed lines of the file:
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@@
-	(wire
-		(pts
-			(xy 22.86 24.13) (xy 24.13 24.13)
-		)
-		(stroke
-			(width 0)
-			(type default)
-		)
-	)
 	(wire
 		(pts
@@
 		)
 	)
-	(label "CS"
-		(at 24.13 24.13 0)
-		(effects
-			(font
-				(size 1.27 1.27)
-			)
-			(justify left bottom)
-		)
-	)
 	(label "SCK"
 		(at 41.91 29.21 180)
@@
 		)
 	)
-	(label "SCK"
+	(label "SDA"
 		(at 24.13 19.05 0)
 		(effects
@@
 		)
 	)
-	(label "MISO"
+	(label "SCL"
 		(at 24.13 21.59 0)
 		(effects
@@
 		)
 	)
-	(hierarchical_label "MISO"
-		(shape input)
+	(hierarchical_label "SCL"
+		(shape bidirectional)
 		(at 22.86 21.59 180)
 		(effects
@@
 		)
 	)
-	(hierarchical_label "CS"
-		(shape input)
-		(at 22.86 24.13 180)
-		(effects
-			(font
-				(size 1.27 1.27)
-			)
-			(justify right)
-		)
-	)
-	(hierarchical_label "SCK"
-		(shape input)
+	(hierarchical_label "SDA"
+		(shape bidirectional)
 		(at 22.86 19.05 180)
 		(effects
@@
 			)
 		)
-		(property "Value" "2x10 Male Pins"
+		(property "Value" "2x18 Male Pins"
 			(at 49.276 17.272 0)
 			(effects
