File: hardware/main_board/main_board.kicad_sch (KiCad schematic)
At the start: 0 parts

Commit message: drew schematic
Other:
- sheet POWER renamed Power
- sheet Encoders & Buttons ports: added ENC1{ENC}, ENC2{ENC}; removed none
- sheet MCU ports: added ENC1{ENC}, ENC2{ENC}; removed none
- sheet Peripheral Boards ports: added none; removed SPI1{SPI}
- note removed: "todo: current budgeting todo: money budgeting"
Changed lines of the file:
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@@
 	(generator_version "9.0")
 	(paper "A4")
-	(text "todo: current budgeting\ntodo: money budgeting"
-		(exclude_from_sim no)
-		(at 53.34 83.82 0)
-		(effects
-			(font
-				(size 1.27 1.27)
-			)
-		)
-	)
-	(junction
-		(at 146.05 116.84)
-		(diameter 0)
-		(color 0 0 0 0)
-	)
 	(bus
 		(pts
@@
 	(wire
 		(pts
-			(xy 138.43 85.09) (xy 158.75 85.09)
+			(xy 138.43 86.36) (xy 158.75 86.36)
 		)
 		(stroke
@@
 	(wire
 		(pts
-			(xy 138.43 82.55) (xy 158.75 82.55)
+			(xy 138.43 83.82) (xy 158.75 83.82)
 		)
 		(stroke
@@
 		)
 	)
+	(bus
+		(pts
+			(xy 146.05 77.47) (xy 146.05 58.42)
+		)
+		(stroke
+			(width 0)
+			(type default)
+		)
+	)
 	(wire
 		(pts
@@
 	(bus
 		(pts
-			(xy 146.05 116.84) (xy 146.05 124.46)
+			(xy 138.43 80.01) (xy 148.59 80.01)
 		)
 		(stroke
@@
 		)
 	)
+	(bus
+		(pts
+			(xy 138.43 77.47) (xy 146.05 77.47)
+		)
+		(stroke
+			(width 0)
+			(type default)
+		)
+	)
 	(wire
 		(pts
@@
 	(bus
 		(pts
+			(xy 146.05 58.42) (xy 158.75 58.42)
+		)
+		(stroke
+			(width 0)
+			(type default)
+		)
+	)
+	(bus
+		(pts
 			(xy 138.43 97.79) (xy 146.05 97.79)
 		)
@@
 		)
 	)
-	(bus
-		(pts
-			(xy 146.05 124.46) (xy 138.43 124.46)
-		)
-		(stroke
-			(width 0)
-			(type default)
-		)
-	)
 	(wire
 		(pts
@@
 		)
 	)
+	(bus
+		(pts
+			(xy 148.59 80.01) (xy 148.59 60.96)
+		)
+		(stroke
+			(width 0)
+			(type default)
+		)
+	)
 	(wire
 		(pts
@@
 		(pts
 			(xy 158.75 110.49) (xy 152.4 110.49)
+		)
+		(stroke
+			(width 0)
+			(type default)
+		)
+	)
+	(bus
+		(pts
+			(xy 148.59 60.96) (xy 158.75 60.96)
 		)
 		(stroke
@@
 		)
 		(pin "ADC_IN" input
-			(at 138.43 82.55 0)
+			(at 138.43 83.82 0)
 			(effects
 				(font
@@
 		)
 		(pin "DAC_OUT" output
-			(at 138.43 85.09 0)
+			(at 138.43 86.36 0)
 			(effects
 				(font
@@
 		(pin "LCD_DC" output
 			(at 138.43 90.17 0)
+			(effects
+				(font
+					(size 1.27 1.27)
+				)
+				(justify right)
+			)
+		)
+		(pin "ENC1{ENC}" output
+			(at 138.43 77.47 0)
+			(effects
+				(font
+					(size 1.27 1.27)
+				)
+				(justify right)
+			)
+		)
+		(pin "ENC2{ENC}" output
+			(at 138.43 80.01 0)
 			(effects
 				(font
@@
 			)
 		)
-		(pin "SPI1{SPI}" input
-			(at 138.43 124.46 0)
-			(effects
-				(font
-					(size 1.27 1.27)
-				)
-				(justify right)
-			)
-		)
 		(pin "S0" input
 			(at 118.11 135.89 180)
@@
 	)
 	(sheet
-		(at 80.01 34.29)
+		(at 118.11 45.72)
 		(size 20.32 21.59)
 		(exclude_from_sim no)
@@
 			(color 0 0 0 0.0000)
 		)
-		(property "Sheetname" "POWER"
-			(at 80.01 33.5784 0)
+		(property "Sheetname" "Power"
+			(at 118.11 45.0084 0)
 			(effects
 				(font
@@
 		)
 		(property "Sheetfile" "POWER.kicad_sch"
-			(at 80.01 56.4646 0)
+			(at 118.11 67.8946 0)
 			(effects
 				(font
@@
 		)
 		(pin "ADC_IN" output
-			(at 158.75 82.55 180)
+			(at 158.75 83.82 180)
 			(effects
 				(font
@@
 		)
 		(pin "DAC_OUT" output
-			(at 158.75 85.09 180)
+			(at 158.75 86.36 180)
 			(effects
 				(font
@@
 			)
 		)
+		(pin "ENC1{ENC}" output
+			(at 158.75 58.42 180)
+			(effects
+				(font
+					(size 1.27 1.27)
+				)
+				(justify left)
+			)
+		)
+		(pin "ENC2{ENC}" output
+			(at 158.75 60.96 180)
+			(effects
+				(font
+					(size 1.27 1.27)
+				)
+				(justify left)
+			)
+		)
 		(instances
 			(project "main_board"
@@
 	)
 	(sheet
-		(at 191.77 104.14)
+		(at 158.75 128.27)
 		(size 20.32 21.59)
 		(exclude_from_sim no)
-		(in_bom yes)
-		(on_board yes)
-		(dnp no)
+		(in_bom no)
+		(on_board no)
+		(dnp yes)
 		(fields_autoplaced yes)
 		(stroke
@@
 		)
 		(property "Sheetname" "LED Strips"
-			(at 191.77 103.4284 0)
+			(at 158.75 127.5584 0)
 			(effects
 				(font
@@
 		)
 		(property "Sheetfile" "LED_STRIPS.kicad_sch"
-			(at 191.77 126.3146 0)
-			(effects
-				(font
+			(at 158.75 150.4446 0)
+			(effects
+				(font

Commit message: save before nuke SPI ADC
Parts:
- added H1, H2, H3, H4, H5: MountingHole, symbol Mechanical:MountingHole
Other:
- sheet Encoders & Buttons ports: added ENC_TOGGLE, ENC{ENC}; removed ENC1{ENC}, ENC2{ENC}
- sheet LCD ports: added CS_LCD, CS_SD; removed CS_{LCD}, CS_{SD}
- sheet MCU ports: added CS_LCD, CS_P[0..4], CS_SD, ENC_TOGGLE, ENC{ENC}, S[0..3]; removed CS_{LCD}, CS_{P1}, CS_{P2}, CS_{P3}, CS_{P4}, CS_{P5}, CS_{SD}, ENC1{ENC}, ENC2{ENC}, S0, S1, S2, S3
- sheet Peripheral Boards ports: added CS_P[0..4], S[0..3]; removed CS_{P1}, CS_{P2}, CS_{P3}, CS_{P4}, CS_{P5}, S0, S1, S2, S3
- note added: "Mounting Holes"

Commit message: port to i2c for both boards. periph board passes drc
Other:
- sheet LCD ports: added SPI0{SPI}; removed SPI1{SPI}
- sheet MCU ports: added I2C0{I2C}; removed CS_P[0..4], SPI1{SPI}
- sheet Peripheral Boards ports: added I2C0{I2C}; removed CS_P[0..4], SPI0{SPI}
Changed lines of the file:
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@@
-		)
-	)
-	(bus
-		(pts
-			(xy 143.51 121.92) (xy 138.43 121.92)
-		)
-		(stroke
-			(width 0)
-			(type default)
 		)
 	)
@@
 		)
 	)
+	(bus
+		(pts
+			(xy 118.11 88.9) (xy 111.76 88.9)
+		)
+		(stroke
+			(width 0)
+			(type default)
+		)
+	)
 	(wire
 		(pts
@@
 		)
 	)
-	(bus
-		(pts
-			(xy 118.11 88.9) (xy 111.76 88.9)
-		)
-		(stroke
-			(width 0)
-			(type default)
-		)
-	)
 	(wire
 		(pts
@@
 	(bus
 		(pts
+			(xy 111.76 132.08) (xy 118.11 132.08)
+		)
+		(stroke
+			(width 0)
+			(type default)
+		)
+	)
+	(wire
+		(pts
+			(xy 152.4 110.49) (xy 152.4 92.71)
+		)
+		(stroke
+			(width 0)
+			(type default)
+		)
+	)
+	(bus
+		(pts
+			(xy 146.05 77.47) (xy 146.05 58.42)
+		)
+		(stroke
+			(width 0)
+			(type default)
+		)
+	)
+	(wire
+		(pts
+			(xy 138.43 86.36) (xy 158.75 86.36)
+		)
+		(stroke
+			(width 0)
+			(type default)
+		)
+	)
+	(bus
+		(pts
 			(xy 111.76 88.9) (xy 111.76 132.08)
 		)
@@
 		)
 	)
-	(wire
-		(pts
-			(xy 152.4 110.49) (xy 152.4 92.71)
-		)
-		(stroke
-			(width 0)
-			(type default)
-		)
-	)
-	(bus
-		(pts
-			(xy 146.05 77.47) (xy 146.05 58.42)
-		)
-		(stroke
-			(width 0)
-			(type default)
-		)
-	)
-	(wire
-		(pts
-			(xy 138.43 86.36) (xy 158.75 86.36)
-		)
-		(stroke
-			(width 0)
-			(type default)
-		)
-	)
-	(bus
-		(pts
-			(xy 138.43 100.33) (xy 143.51 100.33)
-		)
-		(stroke
-			(width 0)
-			(type default)
-		)
-	)
 	(bus
 		(pts
@@
 	(bus
 		(pts
-			(xy 111.76 132.08) (xy 118.11 132.08)
-		)
-		(stroke
-			(width 0)
-			(type default)
-		)
-	)
-	(bus
-		(pts
 			(xy 146.05 58.42) (xy 158.75 58.42)
 		)
@@
 		(pts
 			(xy 149.86 95.25) (xy 149.86 113.03)
-		)
-		(stroke
-			(width 0)
-			(type default)
-		)
-	)
-	(bus
-		(pts
-			(xy 143.51 100.33) (xy 143.51 121.92)
 		)
 		(stroke
@@
 		)
 		(pin "SPI0{SPI}" bidirectional
-			(at 138.43 100.33 0)
-			(effects
-				(font
-					(size 1.27 1.27)
-				)
-				(justify right)
-			)
-		)
-		(pin "SPI1{SPI}" bidirectional
 			(at 138.43 97.79 0)
 			(effects
@@
 			)
 		)
-		(pin "CS_P[0..4]" output
-			(at 118.11 88.9 180)
-			(effects
-				(font
-					(size 1.27 1.27)
-				)
-				(justify left)
-			)
-		)
 		(pin "S[0..3]" output
 			(at 118.11 91.44 180)
@@
 				)
 				(justify right)
+			)
+		)
+		(pin "I2C0{I2C}" bidirectional
+			(at 118.11 88.9 180)
+			(effects
+				(font
+					(size 1.27 1.27)
+				)
+				(justify left)
 			)
 		)
@@
 			)
 		)
-		(pin "SPI0{SPI}" input
-			(at 138.43 121.92 0)
-			(effects
-				(font
-					(size 1.27 1.27)
-				)
-				(justify right)
-			)
-		)
-		(pin "CS_P[0..4]" input
-			(at 118.11 132.08 180)
-			(effects
-				(font
-					(size 1.27 1.27)
-				)
-				(justify left)
-			)
-		)
 		(pin "S[0..3]" input
 			(at 118.11 129.54 180)
+			(effects
+				(font
+					(size 1.27 1.27)
+				)
+				(justify left)
+			)
+		)
+		(pin "I2C0{I2C}" bidirectional
+			(at 118.11 132.08 180)
 			(effects
 				(font
@@
 			)
 		)
-		(pin "SPI1{SPI}" bidirectional
+		(pin "SPI0{SPI}" bidirectional
 			(at 158.75 116.84 180)
 			(effects
