File: hardware/main_board/LED_STRIPS.kicad_sch (KiCad schematic)
At the start: 9 parts, among them IC801 SN74AHCT125DBR, J801 Conn_01x03_Pin, J802 Conn_01x03_Pin

Commit message: finished main pcb
Parts:
- JP801: footprint 445L:PinHeader_1x02_P2.54mm_Vertical -> Jumper:SolderJumper-2_P1.3mm_Open_TrianglePad1.0x1.5mm
- TP801: value LED_D -> DOUT
- TP803: value LED_DATA -> DOUT3V3
Connections:
- net LED_D renamed DOUT
- net LED_DATA* renamed DOUT_5V
Changed lines of the file:
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@@
 	(wire
 		(pts
-			(xy 33.02 20.32) (xy 34.29 20.32)
+			(xy 29.21 21.59) (xy 30.48 21.59)
 		)
 		(stroke
@@
 		)
 	)
-	(label "LED_DATA"
-		(at 34.29 20.32 0)
-		(effects
-			(font
-				(size 1.27 1.27)
-			)
-			(justify left bottom)
-		)
-	)
-	(label "LED_DATA"
+	(label "DOUT_3V3"
+		(at 30.48 21.59 0)
+		(effects
+			(font
+				(size 1.27 1.27)
+			)
+			(justify left bottom)
+		)
+	)
+	(label "DOUT_3V3"
 		(at 59.69 52.07 0)
 		(effects
@@
 		)
 	)
-	(label "LED_DATA*"
+	(label "DOUT_5V"
 		(at 36.83 91.44 0)
 		(effects
@@
 		)
 	)
-	(label "LED_D"
+	(label "DOUT"
 		(at 36.83 88.9 0)
 		(effects
@@
 		)
 	)
-	(label "LED_D"
+	(label "DOUT"
 		(at 40.64 73.66 0)
 		(effects
@@
 		)
 	)
-	(label "LED_DATA"
+	(label "DOUT_3V3"
 		(at 36.83 86.36 0)
 		(effects
@@
 		)
 	)
-	(label "LED_DATA*"
+	(label "DOUT_5V"
 		(at 59.69 54.61 0)
 		(effects
@@
 	(hierarchical_label "LED_DATA"
 		(shape input)
-		(at 33.02 20.32 180)
+		(at 29.21 21.59 180)
 		(effects
 			(font
@@
 			)
 		)
-		(property "Footprint" "445L:PinHeader_1x02_P2.54mm_Vertical"
+		(property "Footprint" "Jumper:SolderJumper-2_P1.3mm_Open_TrianglePad1.0x1.5mm"
 			(at 46.99 76.2 0)
 			(effects
@@
 			)
 		)
-		(property "Value" "LED_D"
+		(property "Value" "DOUT"
 			(at 38.1 69.596 0)
 			(effects
@@
 			)
 		)
-		(property "Value" "LED_DATA"
+		(property "Value" "DOUT3V3"
 			(at 81.026 60.706 0)
 			(effects
